Commit message: update robot urdf file

File: src/spir_description/urdf/solar_panel_installation_robot.urdf (robot description, URDF)
Before this commit: robot solar_panel_installation_robot, 7 links, 6 joints
Links:
- added link camera_optical_frame, mass 1161.6695731136
- link Link_1: mass 1366.3 -> 1161.6695731136
- link Link_2: mass 1366.3 -> 1161.6695731136
- link Link_3: mass 1366.3 -> 1161.6695731136
- link Link_4: mass 1366.3 -> 1161.6695731136
- link Link_5: mass 1366.3 -> 1161.6695731136
- link Link_6: mass 3 -> 44.7597449842918
- link base_link: mass 1366.3 -> 1161.6695731136
Joints:
- removed joint axis-6
- added joint Joint_camera: type fixed, parent Link_6, child camera_optical_frame, origin xyz=0.2444 -0.715 0.0050661 rpy=-1.5705 0 -1.5708, axis 0 0 0
- added joint axis-0: type revolute, parent base_link, child Link_1, origin xyz=0 0 0.2785 rpy=0 0 0, axis 0 0 1, limit lower=-3.1415 upper=3.1415 effort=10 velocity=10
- joint axis-1: axis 0 0 1 -> 0 -1 0; child Link_1 -> Link_2; origin xyz=-1.7894E-05 0 0.2785 rpy=0 0 0 -> xyz=0.400000000000002 0.1345 0.322999999999998 rpy=0 0 0; parent base_link -> Link_1
- joint axis-2: child Link_2 -> Link_3; origin xyz=0.4 0.1345 0.323 rpy=0 0 0 -> xyz=0 -0.00100000000000011 1.20000000000002 rpy=0 0 0; parent Link_1 -> Link_2
- joint axis-3: axis 0 1 0 -> -1 0 -0.00027033; child Link_3 -> Link_4; origin xyz=0 0.029 1.2 rpy=0 0 0 -> xyz=0.39453 -0.26 0.25011 rpy=0 0 0; parent Link_2 -> Link_3
- joint axis-4: axis -1 0 0 -> 0 1 0; child Link_4 -> Link_5; origin xyz=0.39453 -0.29 0.25011 rpy=0 -0.00027033 0 -> xyz=1.2526 -0.168 0.00033861 rpy=0 0 0; parent Link_3 -> Link_4
- joint axis-5: axis 0 1 0 -> -1 0 -0.00027033; child Link_5 -> Link_6; origin xyz=1.2526 -0.15441 -0.015677 rpy=0.10118 0 0 -> xyz=0.277 0.168 7.4881E-05 rpy=0 0 0; parent Link_4 -> Link_5
