Commit message: feat: target sending and command feedback

File: src/spir_description/urdf/spir_description.urdf (robot description, URDF)
Before this commit: robot solar_panel_installation_robot, 8 links, 7 joints
Links:
- removed link camera_optical_frame
Joints:
- removed joint Joint_camera
- joint axis-1: origin xyz=0.400000000000002 0.1345 0.322999999999998 rpy=0 0 0 -> xyz=0.4 0.1345 0.323 rpy=0 0 0
- joint axis-2: origin xyz=0 -0.00100000000000011 1.20000000000002 rpy=0 0 0 -> xyz=0 -0.001 1.2 rpy=0 0 0
- joint axis-3: axis -1 0 -0.00027033 -> -0.99999996346114 0 -0.000270328906909661; origin xyz=0.39453 -0.26 0.25011 rpy=0 0 0 -> xyz=0.394532403355045 -0.259999999999995 0.250106662651998 rpy=0 0 0
